File: CamAdapter/CamAdapter.brd (EAGLE design)
At the start: 22.5 x 41.9 mm, 3 parts

Commit message: Board updates + gcode
Routing:
- net RESET#: track 32.1 -> 33.9 mm
- net CE#: track 35.0 -> 34.5 mm
Changed lines of the file:
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@@
 <contactref element="SV2" pad="2"/>
 <contactref element="SV1" pad="1"/>
-<wire x1="16.51" y1="6.35" x2="17.78" y2="6.35" width="0.4064" layer="16"/>
-<wire x1="17.78" y1="6.35" x2="19.05" y2="7.62" width="0.4064" layer="16"/>
-<wire x1="19.05" y1="7.62" x2="19.05" y2="33.02" width="0.4064" layer="16"/>
-<wire x1="19.05" y1="33.02" x2="16.51" y2="35.56" width="0.4064" layer="16"/>
+<wire x1="16.51" y1="6.35" x2="19.05" y2="6.35" width="0.4064" layer="16"/>
+<wire x1="19.05" y1="6.35" x2="20.32" y2="7.62" width="0.4064" layer="16"/>
+<wire x1="20.32" y1="7.62" x2="20.32" y2="31.75" width="0.4064" layer="16"/>
+<wire x1="20.32" y1="31.75" x2="16.51" y2="35.56" width="0.4064" layer="16"/>
 </signal>
 <signal name="CLK">
@@
 <contactref element="SV1" pad="5"/>
 <wire x1="11.43" y1="6.35" x2="12.7" y2="7.62" width="0.4064" layer="16"/>
-<wire x1="12.7" y1="7.62" x2="12.7" y2="9.525" width="0.4064" layer="16"/>
-<wire x1="12.7" y1="9.525" x2="5.715" y2="16.51" width="0.4064" layer="16"/>
-<wire x1="5.715" y1="16.51" x2="5.715" y2="28.575" width="0.4064" layer="16"/>
-<wire x1="5.715" y1="28.575" x2="11.43" y2="34.29" width="0.4064" layer="16"/>
-<wire x1="11.43" y1="34.29" x2="11.43" y2="35.56" width="0.4064" layer="16"/>
+<wire x1="12.7" y1="7.62" x2="12.7" y2="11.43" width="0.4064" layer="16"/>
+<wire x1="12.7" y1="11.43" x2="6.35" y2="17.78" width="0.4064" layer="16"/>
+<wire x1="6.35" y1="17.78" x2="6.35" y2="27.94" width="0.4064" layer="16"/>
+<wire x1="6.35" y1="27.94" x2="11.43" y2="33.02" width="0.4064" layer="16"/>
+<wire x1="11.43" y1="33.02" x2="11.43" y2="35.56" width="0.4064" layer="16"/>
 </signal>
 <signal name="GND">
@@
 <contactref element="SV2" pad="8"/>
 <contactref element="SV2" pad="9"/>
-<polygon width="0.4064" layer="16" orphans="yes">
+<polygon width="0.4064" layer="16">
 <vertex x="0" y="41.91"/>
 <vertex x="22.86" y="41.91"/>
