File: WiiIR/WiiIr.brd (EAGLE design)
At the start: 54.3 x 74.9 mm, 20 parts

Commit message: XMC Shield servo caps
Parts:
- added C1: 100u, resistor:E2,5-7
- added C2: 100n, resistor:C050-024X044
- moved MOTOR 7.62 mm to (10.2, 66.0)
- moved SERVO 7.62 mm to (17.8, 66.0)
Connections:
- net +5V: now also C1.+, C2.1
- net GND: now also C1.-, C2.2
Routing:
- net +5V: track 56.5 -> 71.7 mm
- net P1.1: track 52.8 -> 57.7 mm
- net P1.2: track 54.5 -> 50.2 mm
Changed lines of the file:
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@@
 <attribute name="OC_FARNELL" value="unknown" x="29.21" y="52.07" size="1.778" layer="27" display="off"/>
 </element>
-<element name="MOTOR" library="con-lstb" package="MA03-1" value="" x="17.78" y="66.04" rot="R270">
+<element name="MOTOR" library="con-lstb" package="MA03-1" value="" x="10.16" y="66.04" rot="R270">
+<attribute name="OC_NEWARK" value="unknown" x="10.16" y="66.04" size="1.778" layer="27" rot="R270" display="off"/>
+<attribute name="MPN" value="" x="10.16" y="66.04" size="1.778" layer="27" rot="R270" display="off"/>
+<attribute name="MF" value="" x="10.16" y="66.04" size="1.778" layer="27" rot="R270" display="off"/>
+<attribute name="OC_FARNELL" value="unknown" x="10.16" y="66.04" size="1.778" layer="27" rot="R270" display="off"/>
+</element>
+<element name="SERVO" library="con-lstb" package="MA03-1" value="" x="17.78" y="66.04" rot="R270">
 <attribute name="OC_NEWARK" value="unknown" x="17.78" y="66.04" size="1.778" layer="27" rot="R270" display="off"/>
 <attribute name="MPN" value="" x="17.78" y="66.04" size="1.778" layer="27" rot="R270" display="off"/>
 <attribute name="MF" value="" x="17.78" y="66.04" size="1.778" layer="27" rot="R270" display="off"/>
 <attribute name="OC_FARNELL" value="unknown" x="17.78" y="66.04" size="1.778" layer="27" rot="R270" display="off"/>
-</element>
-<element name="SERVO" library="con-lstb" package="MA03-1" value="" x="10.16" y="66.04" rot="R270">
-<attribute name="OC_NEWARK" value="unknown" x="10.16" y="66.04" size="1.778" layer="27" rot="R270" display="off"/>
-<attribute name="MPN" value="" x="10.16" y="66.04" size="1.778" layer="27" rot="R270" display="off"/>
-<attribute name="MF" value="" x="10.16" y="66.04" size="1.778" layer="27" rot="R270" display="off"/>
-<attribute name="OC_FARNELL" value="unknown" x="10.16" y="66.04" size="1.778" layer="27" rot="R270" display="off"/>
 </element>
 <element name="BLUETOOTH" library="con-lsta" package="FE07" value="" x="26.67" y="11.43">
@@
 <element name="U$1" library="holes" package="3,0" value="" x="5.08" y="5.08"/>
 <element name="U$2" library="holes" package="3,0" value="" x="49.53" y="66.04"/>
+<element name="C1" library="resistor" package="E2,5-7" value="100u" x="30.48" y="67.31" rot="R90"/>
+<element name="C2" library="resistor" package="C050-024X044" value="100n" x="24.13" y="63.5" rot="R270"/>
 </elements>
 <signals>
@@
 <wire x1="49.53" y1="59.69" x2="46.99" y2="59.69" width="0.8128" layer="16"/>
 <wire x1="46.99" y1="59.69" x2="40.64" y2="66.04" width="0.8128" layer="16"/>
-<wire x1="40.64" y1="66.04" x2="17.78" y2="66.04" width="0.8128" layer="16"/>
+<wire x1="40.64" y1="66.04" x2="10.16" y2="66.04" width="0.8128" layer="16"/>
 <wire x1="3.81" y1="59.69" x2="6.35" y2="59.69" width="0.8128" layer="16"/>
-<wire x1="10.16" y1="66.04" x2="5.08" y2="66.04" width="0.8128" layer="16"/>
+<wire x1="17.78" y1="66.04" x2="5.08" y2="66.04" width="0.8128" layer="16"/>
 <wire x1="5.08" y1="66.04" x2="3.81" y2="64.77" width="0.8128" layer="16"/>
 <wire x1="3.81" y1="64.77" x2="3.81" y2="59.69" width="0.8128" layer="16"/>
-<wire x1="10.16" y1="66.04" x2="17.78" y2="66.04" width="0.8128" layer="16"/>
+<wire x1="17.78" y1="66.04" x2="10.16" y2="66.04" width="0.8128" layer="16"/>
+<contactref element="C1" pad="+"/>
+<contactref element="C2" pad="1"/>
+<wire x1="24.13" y1="66.04" x2="30.48" y2="66.04" width="0" layer="19" extent="1-1"/>
+<wire x1="17.78" y1="66.04" x2="24.13" y2="66.04" width="0" layer="19" extent="1-1"/>
 </signal>
 <signal name="GND">
@@
 <contactref element="BLUETOOTH" pad="1"/>
 <contactref element="DBG_R" pad="1"/>
+<contactref element="C1" pad="-"/>
+<contactref element="C2" pad="2"/>
 </signal>
 <signal name="P2.1">
@@
 <contactref element="SV2" pad="19"/>
 <contactref element="SERVO" pad="3"/>
-<wire x1="46.99" y1="34.29" x2="29.845" y2="34.29" width="0.4064" layer="16"/>
-<wire x1="29.845" y1="34.29" x2="20.32" y2="43.815" width="0.4064" layer="16"/>
-<wire x1="20.32" y1="43.815" x2="20.32" y2="50.8" width="0.4064" layer="16"/>
-<wire x1="20.32" y1="50.8" x2="10.16" y2="60.96" width="0.4064" layer="16"/>
-<wire x1="10.16" y1="60.96" x2="10.16" y2="63.5" width="0.4064" layer="16"/>
+<wire x1="46.99" y1="34.29" x2="31.75" y2="34.29" width="0.4064" layer="16"/>
+<wire x1="31.75" y1="34.29" x2="21.59" y2="44.45" width="0.4064" layer="16"/>
+<wire x1="21.59" y1="44.45" x2="21.59" y2="55.88" width="0.4064" layer="16"/>
+<wire x1="21.59" y1="55.88" x2="17.78" y2="59.69" width="0.4064" layer="16"/>
+<wire x1="17.78" y1="59.69" x2="17.78" y2="63.5" width="0.4064" layer="16"/>
 </signal>
 <signal name="P1.0">
@@
 <contactref element="SV2" pad="20"/>
 <contactref element="MOTOR" pad="3"/>
-<wire x1="49.53" y1="34.29" x2="48.26" y2="35.56" width="0.4064" layer="16"/>
-<wire x1="48.26" y1="35.56" x2="30.48" y2="35.56" width="0.4064" layer="16"/>
-<wire x1="30.48" y1="35.56" x2="21.59" y2="44.45" width="0.4064" layer="16"/>
-<wire x1="21.59" y1="44.45" x2="21.59" y2="52.07" width="0.4064" layer="16"/>
-<wire x1="21.59" y1="52.07" x2="17.78" y2="55.88" width="0.4064" layer="16"/>
-<wire x1="17.78" y1="55.88" x2="17.78" y2="63.5" width="0.4064" layer="16"/>
+<wire x1="49.53" y1="34.29" x2="48.26" y2="33.02" width="0.4064" layer="16"/>
+<wire x1="48.26" y1="33.02" x2="31.75" y2="33.02" width="0.4064" layer="16"/>
+<wire x1="31.75" y1="33.02" x2="20.32" y2="44.45" width="0.4064" layer="16"/>
+<wire x1="20.32" y1="44.45" x2="20.32" y2="49.53" width="0.4064" layer="16"/>
+<wire x1="20.32" y1="49.53" x2="10.16" y2="59.69" width="0.4064" layer="16"/>
+<wire x1="10.16" y1="59.69" x2="10.16" y2="63.5" width="0.4064" layer="16"/>
 </signal>
 <signal name="P1.9">

Commit message: Bent pin headers for servo
Parts:
- MOTOR, SERVO: device con-lstb:MA03-1 -> pinhead:1X03/90
- moved C2 3.59 mm to (26.7, 66.0)
- moved SERVO 3.59 mm to (20.3, 68.6), turned to 0 degrees
- moved C1 2.54 mm to (33.0, 67.3), turned to 270 degrees
- moved MOTOR 2.54 mm to (10.2, 68.6), turned to 0 degrees
Connections:
- net GND: now also MOTOR.3, SERVO.3; no longer MOTOR.1, SERVO.1
- net P1.1: now also MOTOR.1; no longer MOTOR.3
- net P1.2: now also SERVO.1; no longer SERVO.3
Routing:
- net +5V: track 71.7 -> 66.2 mm
- net P1.1: track 57.7 -> 60.1 mm
- net P1.2: track 50.2 -> 51.5 mm
Changed lines of the file:
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@@
 <attribute name="OC_FARNELL" value="unknown" x="29.21" y="52.07" size="1.778" layer="27" display="off"/>
-</element>
-<element name="MOTOR" library="con-lstb" package="MA03-1" value="" x="10.16" y="66.04" rot="R270">
-<attribute name="OC_NEWARK" value="unknown" x="10.16" y="66.04" size="1.778" layer="27" rot="R270" display="off"/>
-<attribute name="MPN" value="" x="10.16" y="66.04" size="1.778" layer="27" rot="R270" display="off"/>
-<attribute name="MF" value="" x="10.16" y="66.04" size="1.778" layer="27" rot="R270" display="off"/>
-<attribute name="OC_FARNELL" value="unknown" x="10.16" y="66.04" size="1.778" layer="27" rot="R270" display="off"/>
-</element>
-<element name="SERVO" library="con-lstb" package="MA03-1" value="" x="17.78" y="66.04" rot="R270">
-<attribute name="OC_NEWARK" value="unknown" x="17.78" y="66.04" size="1.778" layer="27" rot="R270" display="off"/>
-<attribute name="MPN" value="" x="17.78" y="66.04" size="1.778" layer="27" rot="R270" display="off"/>
-<attribute name="MF" value="" x="17.78" y="66.04" size="1.778" layer="27" rot="R270" display="off"/>
-<attribute name="OC_FARNELL" value="unknown" x="17.78" y="66.04" size="1.778" layer="27" rot="R270" display="off"/>
 </element>
 <element name="BLUETOOTH" library="con-lsta" package="FE07" value="" x="26.67" y="11.43">
@@
 <element name="U$1" library="holes" package="3,0" value="" x="5.08" y="5.08"/>
 <element name="U$2" library="holes" package="3,0" value="" x="49.53" y="66.04"/>
-<element name="C1" library="resistor" package="E2,5-7" value="100u" x="30.48" y="67.31" rot="R90"/>
-<element name="C2" library="resistor" package="C050-024X044" value="100n" x="24.13" y="63.5" rot="R270"/>
+<element name="C1" library="resistor" package="E2,5-7" value="100u" x="33.02" y="67.31" rot="R270"/>
+<element name="C2" library="resistor" package="C050-024X044" value="100n" x="26.67" y="66.04" rot="R270"/>
+<element name="MOTOR" library="pinhead" package="1X03/90" value="" x="10.16" y="68.58"/>
+<element name="SERVO" library="pinhead" package="1X03/90" value="" x="20.32" y="68.58"/>
 </elements>
 <signals>
@@
 </signal>
 <signal name="+5V">
-<contactref element="MOTOR" pad="2"/>
-<contactref element="SERVO" pad="2"/>
 <contactref element="SV1" pad="40"/>
 <contactref element="SV1" pad="39"/>
@@
 <contactref element="SV2" pad="40"/>
 <wire x1="49.53" y1="59.69" x2="46.99" y2="59.69" width="0.8128" layer="16"/>
-<wire x1="46.99" y1="59.69" x2="40.64" y2="66.04" width="0.8128" layer="16"/>
-<wire x1="40.64" y1="66.04" x2="10.16" y2="66.04" width="0.8128" layer="16"/>
+<wire x1="46.99" y1="59.69" x2="38.1" y2="68.58" width="0.8128" layer="16"/>
 <wire x1="3.81" y1="59.69" x2="6.35" y2="59.69" width="0.8128" layer="16"/>
-<wire x1="17.78" y1="66.04" x2="5.08" y2="66.04" width="0.8128" layer="16"/>
-<wire x1="5.08" y1="66.04" x2="3.81" y2="64.77" width="0.8128" layer="16"/>
 <wire x1="3.81" y1="64.77" x2="3.81" y2="59.69" width="0.8128" layer="16"/>
-<wire x1="17.78" y1="66.04" x2="10.16" y2="66.04" width="0.8128" layer="16"/>
 <contactref element="C1" pad="+"/>
 <contactref element="C2" pad="1"/>
-<wire x1="24.13" y1="66.04" x2="30.48" y2="66.04" width="0" layer="19" extent="1-1"/>
-<wire x1="17.78" y1="66.04" x2="24.13" y2="66.04" width="0" layer="19" extent="1-1"/>
+<wire x1="3.81" y1="64.77" x2="7.62" y2="68.58" width="0.8128" layer="16"/>
+<wire x1="7.62" y1="68.58" x2="10.16" y2="68.58" width="0.8128" layer="16"/>
+<wire x1="10.16" y1="68.58" x2="20.32" y2="68.58" width="0.8128" layer="16"/>
+<wire x1="20.32" y1="68.58" x2="26.67" y2="68.58" width="0.8128" layer="16"/>
+<wire x1="26.67" y1="68.58" x2="33.02" y2="68.58" width="0.8128" layer="16"/>
+<wire x1="33.02" y1="68.58" x2="38.1" y2="68.58" width="0.8128" layer="16"/>
+<contactref element="MOTOR" pad="2"/>
+<contactref element="SERVO" pad="2"/>
+<wire x1="10.16" y1="64.77" x2="10.16" y2="68.58" width="0.8128" layer="16"/>
+<wire x1="20.32" y1="64.77" x2="20.32" y2="68.58" width="0.8128" layer="16"/>
 </signal>
 <signal name="GND">
@@
 <contactref element="SV2" pad="4"/>
 <contactref element="SV2" pad="36"/>
-<contactref element="MOTOR" pad="1"/>
-<contactref element="SERVO" pad="1"/>
 <contactref element="IR_CAM" pad="9"/>
 <contactref element="IR_CAM" pad="1"/>
@@
 <contactref element="C1" pad="-"/>
 <contactref element="C2" pad="2"/>
+<contactref element="MOTOR" pad="3"/>
+<contactref element="SERVO" pad="3"/>
 </signal>
 <signal name="P2.1">
@@
 <signal name="P1.2">
 <contactref element="SV2" pad="19"/>
-<contactref element="SERVO" pad="3"/>
 <wire x1="46.99" y1="34.29" x2="31.75" y2="34.29" width="0.4064" layer="16"/>
 <wire x1="31.75" y1="34.29" x2="21.59" y2="44.45" width="0.4064" layer="16"/>
 <wire x1="21.59" y1="44.45" x2="21.59" y2="55.88" width="0.4064" layer="16"/>
 <wire x1="21.59" y1="55.88" x2="17.78" y2="59.69" width="0.4064" layer="16"/>
-<wire x1="17.78" y1="59.69" x2="17.78" y2="63.5" width="0.4064" layer="16"/>
+<contactref element="SERVO" pad="1"/>
+<wire x1="17.78" y1="59.69" x2="17.78" y2="64.77" width="0.4064" layer="16"/>
 </signal>
 <signal name="P1.0">
@@
 <signal name="P1.1">
 <contactref element="SV2" pad="20"/>
-<contactref element="MOTOR" pad="3"/>
 <wire x1="49.53" y1="34.29" x2="48.26" y2="33.02" width="0.4064" layer="16"/>
 <wire x1="48.26" y1="33.02" x2="31.75" y2="33.02" width="0.4064" layer="16"/>
 <wire x1="31.75" y1="33.02" x2="20.32" y2="44.45" width="0.4064" layer="16"/>
 <wire x1="20.32" y1="44.45" x2="20.32" y2="49.53" width="0.4064" layer="16"/>
-<wire x1="20.32" y1="49.53" x2="10.16" y2="59.69" width="0.4064" layer="16"/>
-<wire x1="10.16" y1="59.69" x2="10.16" y2="63.5" width="0.4064" layer="16"/>
+<wire x1="20.32" y1="49.53" x2="7.62" y2="62.23" width="0.4064" layer="16"/>
+<contactref element="MOTOR" pad="1"/>
+<wire x1="7.62" y1="62.23" x2="7.62" y2="64.77" width="0.4064" layer="16"/>
 </signal>
 <signal name="P1.9">

Commit message: Board updates + gcode
Other:
- board text added: "Albin F, Christopher G, Matthias Z"
- board text removed: "Albin F., Christopher G., Matthias Z."
Changed lines of the file:
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@@
 <wire x1="54.28" y1="74.92" x2="0" y2="74.92" width="0" layer="20"/>
 <wire x1="0" y1="74.92" x2="0" y2="0" width="0" layer="20"/>
-<text x="52.07" y="71.12" size="1.4224" layer="16" font="vector" ratio="15" rot="MR0">TUtheTOP 2013/14</text>
-<text x="52.07" y="3.81" size="1.4224" layer="16" font="vector" ratio="15" rot="MR0">Albin F., Christopher G., Matthias Z.</text>
+<text x="52.07" y="71.12" size="1.4224" layer="26" font="vector" ratio="20" rot="MR0">TUtheTOP 2013/14</text>
+<text x="52.07" y="3.81" size="1.4224" layer="26" font="vector" ratio="20" rot="MR0">Albin F, Christopher G, Matthias Z</text>
 </plain>
 <attributes>
